Commit message: Renamed realsense packages to avoid name conflicts.

File: realsense2_camera/urdf/_r410.urdf.xacro (robot description, xacro)
@@ -39,5 +39,5 @@
         <geometry>
           <box size="${r410_cam_width} ${r410_cam_height} ${r410_cam_depth}"/>
-          <!--<mesh filename="package://realsense2_camera/meshes/r410/r410.dae" />-->
+          <!--<mesh filename="package://any_realsense2_camera/meshes/r410/r410.dae" />-->
         </geometry>
         <material name="aluminum"/>

File: realsense2_camera/urdf/_r430.urdf.xacro (robot description, xacro)
@@ -40,5 +40,5 @@
         <geometry>
           <box size="${r430_cam_width} ${r430_cam_height} ${r430_cam_depth}"/>
-          <!--<mesh filename="package://realsense2_camera/meshes/r430/r430.dae" />-->
+          <!--<mesh filename="package://any_realsense2_camera/meshes/r430/r430.dae" />-->
         </geometry>
         <material name="aluminum"/>

File: realsense2_camera/urdf/test_r410_camera.urdf.xacro (robot description, xacro)
@@ -1,5 +1,5 @@
 <?xml version="1.0"?>
-<robot name="realsense2_camera" xmlns:xacro="http://ros.org/wiki/xacro">
-  <xacro:include filename="$(find realsense2_camera)/urdf/_r410.urdf.xacro"/>
+<robot name="any_realsense2_camera" xmlns:xacro="http://ros.org/wiki/xacro">
+  <xacro:include filename="$(find any_realsense2_camera)/urdf/_r410.urdf.xacro"/>
   <link name="base_link" />
   <sensor_r410 parent="base_link">

File: realsense2_camera/urdf/test_r430_camera.urdf.xacro (robot description, xacro)
@@ -1,5 +1,5 @@
 <?xml version="1.0"?>
-<robot name="realsense2_camera" xmlns:xacro="http://ros.org/wiki/xacro">
-  <xacro:include filename="$(find realsense2_camera)/urdf/_r430.urdf.xacro"/>
+<robot name="any_realsense2_camera" xmlns:xacro="http://ros.org/wiki/xacro">
+  <xacro:include filename="$(find any_realsense2_camera)/urdf/_r430.urdf.xacro"/>
   <link name="base_link" />
   <sensor_r430 parent="base_link">

Commit message: Reverted renaming.

File: realsense2_camera/urdf/_r410.urdf.xacro (robot description, xacro)
@@ -39,5 +39,5 @@
         <geometry>
           <box size="${r410_cam_width} ${r410_cam_height} ${r410_cam_depth}"/>
-          <!--<mesh filename="package://any_realsense2_camera/meshes/r410/r410.dae" />-->
+          <!--<mesh filename="package://realsense2_camera/meshes/r410/r410.dae" />-->
         </geometry>
         <material name="aluminum"/>

File: realsense2_camera/urdf/_r430.urdf.xacro (robot description, xacro)
@@ -40,5 +40,5 @@
         <geometry>
           <box size="${r430_cam_width} ${r430_cam_height} ${r430_cam_depth}"/>
-          <!--<mesh filename="package://any_realsense2_camera/meshes/r430/r430.dae" />-->
+          <!--<mesh filename="package://realsense2_camera/meshes/r430/r430.dae" />-->
         </geometry>
         <material name="aluminum"/>

File: realsense2_camera/urdf/test_r410_camera.urdf.xacro (robot description, xacro)
@@ -1,5 +1,5 @@
 <?xml version="1.0"?>
-<robot name="any_realsense2_camera" xmlns:xacro="http://ros.org/wiki/xacro">
-  <xacro:include filename="$(find any_realsense2_camera)/urdf/_r410.urdf.xacro"/>
+<robot name="realsense2_camera" xmlns:xacro="http://ros.org/wiki/xacro">
+  <xacro:include filename="$(find realsense2_camera)/urdf/_r410.urdf.xacro"/>
   <link name="base_link" />
   <sensor_r410 parent="base_link">

File: realsense2_camera/urdf/test_r430_camera.urdf.xacro (robot description, xacro)
@@ -1,5 +1,5 @@
 <?xml version="1.0"?>
-<robot name="any_realsense2_camera" xmlns:xacro="http://ros.org/wiki/xacro">
-  <xacro:include filename="$(find any_realsense2_camera)/urdf/_r430.urdf.xacro"/>
+<robot name="realsense2_camera" xmlns:xacro="http://ros.org/wiki/xacro">
+  <xacro:include filename="$(find realsense2_camera)/urdf/_r430.urdf.xacro"/>
   <link name="base_link" />
   <sensor_r430 parent="base_link">
